File: KiCad/pcb-dev-fpga-iCE40/Memory.sch (KiCad schematic (older format))
At the start: 8 parts, among them U2 LY68L6400, U3 W25Q128JVxxM

Commit message: Assign footprints
Parts:
- C14: footprint (none) -> Capacitor_SMD:C_0603_1608Metric
- JP5, JP6: footprint (none) -> Jumper:SolderJumper-2_P1.3mm_Open_Pad1.0x1.5mm
- R10, R8, R9: footprint (none) -> Resistor_SMD:R_0603_1608Metric
- U2: footprint (none) -> LY68L6400:SOIC127P600X175-8N
- U3: footprint (none) -> W25Q128JVx:SOIC127P1032X264-16N
Changed lines of the file:
@@
 F 0 "U2" H 4600 3825 50  0000 C CNN
 F 1 "LY68L6400" H 4600 3734 50  0000 C CNN
-F 2 "" H 4600 3300 50  0001 C CNN
+F 2 "LY68L6400:SOIC127P600X175-8N" H 4600 3300 50  0001 C CNN
 F 3 "" H 4600 3300 50  0001 C CNN
 	1    4600 3300
@@
 F 0 "U3" H 4600 4825 50  0000 C CNN
 F 1 "W25Q128JVxxM" H 4600 4734 50  0000 C CNN
-F 2 "" H 4800 4400 50  0001 C CNN
+F 2 "W25Q128JVx:SOIC127P1032X264-16N" H 4800 4400 50  0001 C CNN
 F 3 "" H 4800 4400 50  0001 C CNN
 	1    4600 4400
@@
 F 0 "C14" H 3650 4350 50  0000 L CNN
 F 1 "100n" H 3600 4250 50  0000 L CNN
-F 2 "" H 3900 4300 50  0001 C CNN
+F 2 "Capacitor_SMD:C_0603_1608Metric" H 3900 4300 50  0001 C CNN
 F 3 "~" H 3900 4300 50  0001 C CNN
 	1    3900 4300
@@
 F 0 "JP5" H 7150 3185 50  0000 C CNN
 F 1 "Jumper" H 7150 3094 50  0000 C CNN
-F 2 "" H 7150 3000 50  0001 C CNN
+F 2 "Jumper:SolderJumper-2_P1.3mm_Open_Pad1.0x1.5mm" H 7150 3000 50  0001 C CNN
 F 3 "~" H 7150 3000 50  0001 C CNN
 	1    7150 3000
@@
 F 0 "JP6" H 7150 4385 50  0000 C CNN
 F 1 "Jumper" H 7150 4294 50  0000 C CNN
-F 2 "" H 7150 4200 50  0001 C CNN
+F 2 "Jumper:SolderJumper-2_P1.3mm_Open_Pad1.0x1.5mm" H 7150 4200 50  0001 C CNN
 F 3 "~" H 7150 4200 50  0001 C CNN
 	1    7150 4200
@@
 F 0 "R8" H 5909 2796 50  0000 L CNN
 F 1 "10k" H 5909 2705 50  0000 L CNN
-F 2 "" H 5850 2750 50  0001 C CNN
+F 2 "Resistor_SMD:R_0603_1608Metric" H 5850 2750 50  0001 C CNN
 F 3 "~" H 5850 2750 50  0001 C CNN
 	1    5850 2750
@@
 F 0 "R9" H 6159 2796 50  0000 L CNN
 F 1 "10k" H 6159 2705 50  0000 L CNN
-F 2 "" H 6100 2750 50  0001 C CNN
+F 2 "Resistor_SMD:R_0603_1608Metric" H 6100 2750 50  0001 C CNN
 F 3 "~" H 6100 2750 50  0001 C CNN
 	1    6100 2750
@@
 F 0 "R10" H 6409 2796 50  0000 L CNN
 F 1 "10k" H 6409 2705 50  0000 L CNN
-F 2 "" H 6350 2750 50  0001 C CNN
+F 2 "Resistor_SMD:R_0603_1608Metric" H 6350 2750 50  0001 C CNN
 F 3 "~" H 6350 2750 50  0001 C CNN
 	1    6350 2750
