File: KiCad/pcb-dev-fpga-iCE40/Power.sch (KiCad schematic (older format))
At the start: 8 parts, among them U4 TLV75533PDRV, U5 TLV73312PDBV

Commit message: Assign footprints
Parts:
- C15, C16, C17, C18, C19: footprint (none) -> Capacitor_SMD:C_0603_1608Metric
- R11: footprint (none) -> Resistor_SMD:R_0603_1608Metric
Changed lines of the file:
@@
 F 0 "R11" H 4041 3654 50  0000 R CNN
 F 1 "10k" H 4041 3745 50  0000 R CNN
-F 2 "" H 4100 3700 50  0001 C CNN
+F 2 "Resistor_SMD:R_0603_1608Metric" H 4100 3700 50  0001 C CNN
 F 3 "~" H 4100 3700 50  0001 C CNN
 	1    4100 3700
@@
 F 0 "C15" H 4192 4146 50  0000 L CNN
 F 1 "1u" H 4192 4055 50  0000 L CNN
-F 2 "" H 4100 4100 50  0001 C CNN
+F 2 "Capacitor_SMD:C_0603_1608Metric" H 4100 4100 50  0001 C CNN
 F 3 "~" H 4100 4100 50  0001 C CNN
 	1    4100 4100
@@
 F 0 "C16" H 4442 4146 50  0000 L CNN
 F 1 "4u7" H 4442 4055 50  0000 L CNN
-F 2 "" H 4350 4100 50  0001 C CNN
+F 2 "Capacitor_SMD:C_0603_1608Metric" H 4350 4100 50  0001 C CNN
 F 3 "~" H 4350 4100 50  0001 C CNN
 	1    4350 4100
@@
 F 0 "C17" H 5342 4046 50  0000 L CNN
 F 1 "4u7" H 5342 3955 50  0000 L CNN
-F 2 "" H 5250 4000 50  0001 C CNN
+F 2 "Capacitor_SMD:C_0603_1608Metric" H 5250 4000 50  0001 C CNN
 F 3 "~" H 5250 4000 50  0001 C CNN
 	1    5250 4000
@@
 F 0 "C18" H 6642 4046 50  0000 L CNN
 F 1 "4u7" H 6642 3955 50  0000 L CNN
-F 2 "" H 6550 4000 50  0001 C CNN
+F 2 "Capacitor_SMD:C_0603_1608Metric" H 6550 4000 50  0001 C CNN
 F 3 "~" H 6550 4000 50  0001 C CNN
 	1    6550 4000
@@
 F 0 "C19" H 7642 4046 50  0000 L CNN
 F 1 "4u7" H 7642 3955 50  0000 L CNN
-F 2 "" H 7550 4000 50  0001 C CNN
+F 2 "Capacitor_SMD:C_0603_1608Metric" H 7550 4000 50  0001 C CNN
 F 3 "~" H 7550 4000 50  0001 C CNN
 	1    7550 4000
