File: KiCad/pcb-dev-fpga-iCE40/USB.sch (KiCad schematic (older format))
At the start: 8 parts, among them J3 USB-C Receptacle (USB2.0), U6 USBLC6-2P6

Commit message: Assign footprints
Parts:
- J3: footprint (none) -> USB-C Receptacle:632723300021
- JP7: footprint (none) -> Jumper:SolderJumper-2_P1.3mm_Open_Pad1.0x1.5mm
- R12, R13, R14, R15, R16: footprint (none) -> Resistor_SMD:R_0603_1608Metric
Changed lines of the file:
@@
 F 0 "J3" H 4507 4767 50  0000 C CNN
 F 1 "USB-C Receptacle (USB2.0)" H 4507 4676 50  0000 C CNN
-F 2 "" H 4550 3900 50  0001 C CNN
+F 2 "USB-C Receptacle:632723300021" H 4550 3900 50  0001 C CNN
 F 3 "https://www.usb.org/sites/default/files/documents/usb_type-c.zip" H 4550 3900 50  0001 C CNN
 	1    4400 3900
@@
 F 0 "R12" V 5250 3350 50  0000 C CNN
 F 1 "5k1" V 5250 3700 50  0000 C CNN
-F 2 "" H 5300 3500 50  0001 C CNN
+F 2 "Resistor_SMD:R_0603_1608Metric" H 5300 3500 50  0001 C CNN
 F 3 "~" H 5300 3500 50  0001 C CNN
 	1    5300 3500
@@
 F 0 "R13" V 5250 3450 50  0000 C CNN
 F 1 "5k1" V 5250 3800 50  0000 C CNN
-F 2 "" H 5300 3600 50  0001 C CNN
+F 2 "Resistor_SMD:R_0603_1608Metric" H 5300 3600 50  0001 C CNN
 F 3 "~" H 5300 3600 50  0001 C CNN
 	1    5300 3600
@@
 F 0 "JP7" V 5254 3148 50  0000 L CNN
 F 1 "Jumper" V 5345 3148 50  0000 L CNN
-F 2 "" H 5300 3100 50  0001 C CNN
+F 2 "Jumper:SolderJumper-2_P1.3mm_Open_Pad1.0x1.5mm" H 5300 3100 50  0001 C CNN
 F 3 "~" H 5300 3100 50  0001 C CNN
 	1    5300 3100
@@
 F 0 "R15" V 7304 3750 50  0000 C CNN
 F 1 "22e" V 7395 3750 50  0000 C CNN
-F 2 "" H 7500 3750 50  0001 C CNN
+F 2 "Resistor_SMD:R_0603_1608Metric" H 7500 3750 50  0001 C CNN
 F 3 "~" H 7500 3750 50  0001 C CNN
 	1    7500 3750
@@
 F 0 "R16" V 7304 4050 50  0000 C CNN
 F 1 "22e" V 7395 4050 50  0000 C CNN
-F 2 "" H 7500 4050 50  0001 C CNN
+F 2 "Resistor_SMD:R_0603_1608Metric" H 7500 4050 50  0001 C CNN
 F 3 "~" H 7500 4050 50  0001 C CNN
 	1    7500 4050
@@
 F 0 "R14" H 7050 4200 50  0000 L CNN
 F 1 "1k5" H 7000 4100 50  0000 L CNN
-F 2 "" H 7200 4150 50  0001 C CNN
+F 2 "Resistor_SMD:R_0603_1608Metric" H 7200 4150 50  0001 C CNN
 F 3 "~" H 7200 4150 50  0001 C CNN
 	1    7200 4150
