File: KiCad/pcb-dev-fpga-iCE40/pcb-dev-fpga-iCE40.sch (KiCad schematic (older format))
At the start: 0 parts

Commit message: Add library symbols, finish schematics and export PDF
Parts:
- added C1, C11, C12, C2, C3, C4, C6, C7: 100n, symbol Device:C_Small
- added C10: 10u, symbol Device:C_Small
- added C13, C8: 10n, symbol Device:C_Small
- added C5, C9: 1u, symbol Device:C_Small
- added D1: RED_LED, symbol Device:LED
- added D2: GREEN_LED, symbol Device:LED
- added D3: BLUE_LED, symbol Device:LED
- added D4: RGB LED, symbol Device:LED_RGB
- added J1: Header 1, symbol Connector:Conn_01x20_Female
- added J2: Header 2, symbol Connector:Conn_01x20_Female
- added JP1, JP2, JP3, JP4: Jumper, symbol Device:Jumper_NO_Small
- added R1, R2, R3: 2k2, symbol Device:R_Small
- added R4, R5, R6: 10k, symbol Device:R_Small
- added R7: 100e, symbol Device:R_Small
- added SW1: SPST Switch, symbol Switch:SW_SPST
- added U1: ICE40UP5K-SG48ITR, Package_DFN_QFN:QFN-48-1EP_7x7mm_P0.5mm_EP5.6x5.6mm, symbol FPGA_Lattice:ICE40UP5K-SG48ITR
- added Y1: 12MHz, symbol Device:Crystal_GND24_Small
Connections:
- new net: C1.1, JP1.2, U1.33 (VCCIO_0)
- new net: C3.1, JP2.2, U1.22 (SPI_VCCIO1)
- new net: C4.1, JP3.2, U1.1 (VCCIO_2)
- new net: C6.1, JP4.1, U1.24 (VPP_2V5)
- new net: C10.1, C12.1, R7.2, U1.29 (VCCPLL)
- new net: D1.2 (A), R1.2
- new net: D2.2 (A), R2.2
- new net +1V2: C11.1, C13.1, C5.1, C7.1, C8.1, C9.1, R7.1, U1.30 (VCC), U1.5 (VCC)
- new net +3V3: C2.1, D4.4 (BA), D4.5 (GA), D4.6 (RA), J1.4 (Pin_4), JP1.1, JP2.1, JP3.1, JP4.2, R1.1, R2.1, R3.1, R4.1, R5.1, Y1.4
- new net CDONE: D3.2 (A), R3.2, U1.7 (CDONE)
- new net CLK: U1.35 (IOT_46b_G0), Y1.3
- new net CLK_EN: R5.2, Y1.1
- new net GND: C1.2, C10.2, C11.2, C12.2, C13.2, C2.2, C3.2, C4.2, C5.2, C6.2, C7.2, C8.2, C9.2, D3.1 (K), J1.5 (Pin_5), SW1.1 (A), U1.49 (GND), Y1.2
- new net IOB_0a: J2.14 (Pin_14), U1.46 (IOB_0a)
- new net IOB_13b-~LEDG: D2.1 (K), U1.6 (IOB_13b)
- new net IOB_16a: J2.7 (Pin_7), U1.9 (IOB_16a)
- new net IOB_18a: J2.6 (Pin_6), U1.10 (IOB_18a)
- new net IOB_20a: J2.5 (Pin_5), U1.11 (IOB_20a)
- new net IOB_22b: J2.4 (Pin_4), U1.12 (IOB_22b)
- new net IOB_23b: J2.3 (Pin_3), U1.21 (IOB_23b)
- new net IOB_24a: J2.2 (Pin_2), U1.13 (IOB_24a)
- new net IOB_25b_G3: J2.1 (Pin_1), U1.20 (IOB_25b_G3)
- new net IOB_2a: J2.13 (Pin_13), U1.47 (IOB_2a)
- new net IOB_3b_G6: J2.12 (Pin_12), U1.44 (IOB_3b_G6)
- new net IOB_4a: J2.11 (Pin_11), U1.48 (IOB_4a)
- new net IOB_5b: J2.10 (Pin_10), U1.45 (IOB_5b)
- new net IOB_8a: J2.9 (Pin_9), U1.4 (IOB_8a)
- new net IOB_9b: J2.8 (Pin_8), U1.3 (IOB_9b)
- new net IOT_36b-~LEDR: D1.1 (K), U1.25 (IOT_36b)
- new net IOT_37a: J1.8 (Pin_8), U1.23 (IOT_37a)
- new net IOT_38b: J1.9 (Pin_9), U1.27 (IOT_38b)
- new net IOT_39a: J1.10 (Pin_10), U1.26 (IOT_39a)
- new net IOT_41a: J1.11 (Pin_11), U1.28 (IOT_41a)
- new net IOT_42b: J1.12 (Pin_12), U1.31 (IOT_42b)
- new net IOT_43a: J1.13 (Pin_13), U1.32 (IOT_43a)
- new net IOT_44b: J1.14 (Pin_14), U1.34 (IOT_44b)
- new net IOT_48b: J1.18 (Pin_18), U1.36 (IOT_48b)
- new net IOT_49a: J1.19 (Pin_19), U1.43 (IOT_49a)
- new net SPI_MISO_IO1: J2.18 (Pin_18), U1.17 (IOB_33b_SPI_SI)
- new net SPI_MOSI-IO0: J2.17 (Pin_17), U1.14 (IOB_32a_SPI_SO)
- new net SPI_SCK: J2.16 (Pin_16), U1.15 (IOB_34a_SPI_SCK)
- new net SPI_~CS: J2.15 (Pin_15), U1.16 (IOB_35b_SPI_SS)
- new net SPI_~HLD~-I03: J2.20 (Pin_20), U1.19 (IOB_29b)
- new net SPI_~WP~-I02: J2.19 (Pin_19), U1.18 (IOB_31b)
- new net USB_DET: U1.37 (IOT_45a_G1)
- new net USB_N: U1.38 (IOT_50b)
- new net USB_P: U1.42 (IOT_51a)
- new net VCCIO_2: R6.1
- new net VIN: J1.2 (Pin_2)
- new net ~BTN: R6.2, SW1.2 (B), U1.2 (IOB_6a)
- new net ~CRESET: R4.2, U1.8 (~CRESET)
- new net ~RGB0: D4.1 (RK), U1.39 (RGB0)
- new net ~RGB1: D4.2 (GK), U1.40 (RGB1)
- new net ~RGB2: D4.3 (BK), U1.41 (RGB2)
- no-connect marks 0 -> 8
Other:
- note added: "BUTTON"
- note added: "CLOCK"
- note added: "CONNECTORS"
- note added: "FIELD PROGRAMMABLE GATE ARRAY"
- note added: "FPGA\nDECOUPLING\nCAPACITORS"
- note added: "LEDs"

Commit message: Assign footprints
Parts:
- C1, C10, C11, C12, C13, C2, C3, C4, C5, C6, C7, C8, C9: footprint (none) -> Capacitor_SMD:C_0603_1608Metric
- D1, D2, D3: footprint (none) -> LED_SMD:LED_0603_1608Metric
- D4: footprint (none) -> LED_SMD:LED_RGB_1210
- J1, J2: footprint (none) -> Connector_PinHeader_2.54mm:PinHeader_1x10_P2.54mm_Vertical
- JP1, JP2, JP3, JP4: footprint (none) -> Jumper:SolderJumper-2_P1.3mm_Open_Pad1.0x1.5mm
- R1, R2, R3, R4, R5, R6, R7: footprint (none) -> Resistor_SMD:R_0603_1608Metric
- SW1: footprint (none) -> Button_Switch_SMD:SW_SPST_B3S-1000
- Y1: footprint (none) -> Crystal:Crystal_SMD_0603-4Pin_6.0x3.5mm
Changed lines of the file:
@@
 F 0 "Y1" H 5100 5400 50  0000 L CNN
 F 1 "12MHz" H 5100 5300 50  0000 L CNN
-F 2 "" H 5000 5500 50  0001 C CNN
+F 2 "Crystal:Crystal_SMD_0603-4Pin_6.0x3.5mm" H 5000 5500 50  0001 C CNN
 F 3 "~" H 5000 5500 50  0001 C CNN
 	1    5000 5500
@@
 F 0 "SW1" H 7050 5735 50  0000 C CNN
 F 1 "SPST Switch" H 7050 5644 50  0000 C CNN
-F 2 "" H 7050 5500 50  0001 C CNN
+F 2 "Button_Switch_SMD:SW_SPST_B3S-1000" H 7050 5500 50  0001 C CNN
 F 3 "~" H 7050 5500 50  0001 C CNN
 	1    7050 5500
@@
 F 0 "R6" H 7409 5446 50  0000 L CNN
 F 1 "10k" H 7409 5355 50  0000 L CNN
-F 2 "" H 7350 5400 50  0001 C CNN
+F 2 "Resistor_SMD:R_0603_1608Metric" H 7350 5400 50  0001 C CNN
 F 3 "~" H 7350 5400 50  0001 C CNN
 	1    7350 5400
@@
 F 0 "D1" H 2043 5017 50  0000 C CNN
 F 1 "RED_LED" H 2043 4926 50  0000 C CNN
-F 2 "" H 2050 4800 50  0001 C CNN
+F 2 "LED_SMD:LED_0603_1608Metric" H 2050 4800 50  0001 C CNN
 F 3 "~" H 2050 4800 50  0001 C CNN
 	1    2050 4800
@@
 F 0 "D2" H 2043 5317 50  0000 C CNN
 F 1 "GREEN_LED" H 2043 5226 50  0000 C CNN
-F 2 "" H 2050 5100 50  0001 C CNN
+F 2 "LED_SMD:LED_0603_1608Metric" H 2050 5100 50  0001 C CNN
 F 3 "~" H 2050 5100 50  0001 C CNN
 	1    2050 5100
@@
 F 0 "D3" H 2043 5617 50  0000 C CNN
 F 1 "BLUE_LED" H 2043 5526 50  0000 C CNN
-F 2 "" H 2050 5400 50  0001 C CNN
+F 2 "LED_SMD:LED_0603_1608Metric" H 2050 5400 50  0001 C CNN
 F 3 "~" H 2050 5400 50  0001 C CNN
 	1    2050 5400
@@
 F 0 "R1" V 2204 4800 50  0000 C CNN
 F 1 "2k2" V 2295 4800 50  0000 C CNN
-F 2 "" H 2400 4800 50  0001 C CNN
+F 2 "Resistor_SMD:R_0603_1608Metric" H 2400 4800 50  0001 C CNN
 F 3 "~" H 2400 4800 50  0001 C CNN
 	1    2400 4800
@@
 F 0 "R2" V 2204 5100 50  0000 C CNN
 F 1 "2k2" V 2295 5100 50  0000 C CNN
-F 2 "" H 2400 5100 50  0001 C CNN
+F 2 "Resistor_SMD:R_0603_1608Metric" H 2400 5100 50  0001 C CNN
 F 3 "~" H 2400 5100 50  0001 C CNN
 	1    2400 5100
@@
 F 0 "R3" V 2204 5400 50  0000 C CNN
 F 1 "2k2" V 2295 5400 50  0000 C CNN
-F 2 "" H 2400 5400 50  0001 C CNN
+F 2 "Resistor_SMD:R_0603_1608Metric" H 2400 5400 50  0001 C CNN
 F 3 "~" H 2400 5400 50  0001 C CNN
 	1    2400 5400
@@
 F 0 "D4" H 2050 6497 50  0000 C CNN
 F 1 "RGB LED" H 2050 6406 50  0000 C CNN
-F 2 "" H 2050 5950 50  0001 C CNN
+F 2 "LED_SMD:LED_RGB_1210" H 2050 5950 50  0001 C CNN
 F 3 "~" H 2050 5950 50  0001 C CNN
 	1    2050 6000
@@
 F 0 "C4" H 7742 1996 50  0000 L CNN
 F 1 "100n" H 7742 1905 50  0000 L CNN
-F 2 "" H 7650 1950 50  0001 C CNN
+F 2 "Capacitor_SMD:C_0603_1608Metric" H 7650 1950 50  0001 C CNN
 F 3 "~" H 7650 1950 50  0001 C CNN
 	1    7650 1950
@@
 F 0 "C1" H 2942 1446 50  0000 L CNN
 F 1 "100n" H 2942 1355 50  0000 L CNN
-F 2 "" H 2850 1400 50  0001 C CNN
+F 2 "Capacitor_SMD:C_0603_1608Metric" H 2850 1400 50  0001 C CNN
 F 3 "~" H 2850 1400 50  0001 C CNN
 	1    2850 1400
@@
 F 0 "C3" H 5542 1396 50  0000 L CNN
 F 1 "100n" H 5542 1305 50  0000 L CNN
-F 2 "" H 5450 1350 50  0001 C CNN
+F 2 "Capacitor_SMD:C_0603_1608Metric" H 5450 1350 50  0001 C CNN
 F 3 "~" H 5450 1350 50  0001 C CNN
 	1    5450 1350
@@
 F 0 "J1" H 9800 4250 50  0000 L CNN
 F 1 "Header 1" H 9650 4150 50  0000 L CNN
-F 2 "" H 9950 5300 50  0001 C CNN
+F 2 "Connector_PinHeader_2.54mm:PinHeader_1x10_P2.54mm_Vertical" H 9950 5300 50  0001 C CNN
 F 3 "~" H 9950 5300 50  0001 C CNN
 	1    9950 5300
@@
 F 0 "J2" H 10100 4250 50  0000 C CNN
 F 1 "Header 2" H 10100 4150 50  0000 C CNN
-F 2 "" H 10200 5300 50  0001 C CNN
+F 2 "Connector_PinHeader_2.54mm:PinHeader_1x10_P2.54mm_Vertical" H 10200 5300 50  0001 C CNN
 F 3 "~" H 10200 5300 50  0001 C CNN
 	1    10200 5300
@@
 F 0 "R5" V 4896 5350 50  0000 C CNN
 F 1 "10k" V 4805 5350 50  0000 C CNN
-F 2 "" H 4700 5350 50  0001 C CNN
+F 2 "Resistor_SMD:R_0603_1608Metric" H 4700 5350 50  0001 C CNN
 F 3 "~" H 4700 5350 50  0001 C CNN
 	1    4700 5350
@@
 F 0 "C2" H 4242 5396 50  0000 L CNN
 F 1 "100n" H 4242 5305 50  0000 L CNN
-F 2 "" H 4150 5350 50  0001 C CNN
+F 2 "Capacitor_SMD:C_0603_1608Metric" H 4150 5350 50  0001 C CNN
 F 3 "~" H 4150 5350 50  0001 C CNN
 	1    4150 5350
@@
 F 0 "C5" H 8942 1796 50  0000 L CNN
 F 1 "1u" H 8942 1705 50  0000 L CNN
-F 2 "" H 8850 1750 50  0001 C CNN
+F 2 "Capacitor_SMD:C_0603_1608Metric" H 8850 1750 50  0001 C CNN
 F 3 "~" H 8850 1750 50  0001 C CNN
 	1    8850 1750
@@
 F 0 "C7" H 9242 1796 50  0000 L CNN
 F 1 "100n" H 9242 1705 50  0000 L CNN
-F 2 "" H 9150 1750 50  0001 C CNN
+F 2 "Capacitor_SMD:C_0603_1608Metric" H 9150 1750 50  0001 C CNN
 F 3 "~" H 9150 1750 50  0001 C CNN
 	1    9150 1750
@@
 F 0 "C8" H 9542 1796 50  0000 L CNN
 F 1 "10n" H 9542 1705 50  0000 L CNN
-F 2 "" H 9450 1750 50  0001 C CNN
+F 2 "Capacitor_SMD:C_0603_1608Metric" H 9450 1750 50  0001 C CNN
 F 3 "~" H 9450 1750 50  0001 C CNN
 	1    9450 1750
@@
 F 0 "C9" H 9842 1796 50  0000 L CNN
 F 1 "1u" H 9842 1705 50  0000 L CNN
-F 2 "" H 9750 1750 50  0001 C CNN
+F 2 "Capacitor_SMD:C_0603_1608Metric" H 9750 1750 50  0001 C CNN
 F 3 "~" H 9750 1750 50  0001 C CNN
 	1    9750 1750
@@
 F 0 "C11" H 10142 1796 50  0000 L CNN
 F 1 "100n" H 10142 1705 50  0000 L CNN
-F 2 "" H 10050 1750 50  0001 C CNN
+F 2 "Capacitor_SMD:C_0603_1608Metric" H 10050 1750 50  0001 C CNN
 F 3 "~" H 10050 1750 50  0001 C CNN
 	1    10050 1750
@@
 F 0 "C13" H 10442 1796 50  0000 L CNN
 F 1 "10n" H 10442 1705 50  0000 L CNN
-F 2 "" H 10350 1750 50  0001 C CNN
+F 2 "Capacitor_SMD:C_0603_1608Metric" H 10350 1750 50  0001 C CNN
 F 3 "~" H 10350 1750 50  0001 C CNN
 	1    10350 1750
@@
 F 0 "R7" H 9759 2496 50  0000 L CNN
 F 1 "100e" H 9759 2405 50  0000 L CNN
-F 2 "" H 9700 2450 50  0001 C CNN
+F 2 "Resistor_SMD:R_0603_1608Metric" H 9700 2450 50  0001 C CNN
 F 3 "~" H 9700 2450 50  0001 C CNN
 	1    9700 2450
@@
 F 0 "JP4" V 9550 2600 50  0000 R CNN
 F 1 "Jumper" V 9500 2750 50  0000 R CNN
-F 2 "" H 9500 2450 50  0001 C CNN
+F 2 "Jumper:SolderJumper-2_P1.3mm_Open_Pad1.0x1.5mm" H 9500 2450 50  0001 C CNN
 F 3 "~" H 9500 2450 50  0001 C CNN
 	1    9500 2450
@@
 F 0 "C10" H 10042 3046 50  0000 L CNN
 F 1 "10u" H 10042 2955 50  0000 L CNN
-F 2 "" H 9950 3000 50  0001 C CNN
+F 2 "Capacitor_SMD:C_0603_1608Metric" H 9950 3000 50  0001 C CNN
 F 3 "~" H 9950 3000 50  0001 C CNN
 	1    9950 3000
@@
 F 0 "C12" H 10342 3046 50  0000 L CNN
 F 1 "100n" H 10342 2955 50  0000 L CNN
-F 2 "" H 10250 3000 50  0001 C CNN
+F 2 "Capacitor_SMD:C_0603_1608Metric" H 10250 3000 50  0001 C CNN
 F 3 "~" H 10250 3000 50  0001 C CNN
 	1    10250 3000
@@
 F 0 "C6" H 9192 3046 50  0000 L CNN
 F 1 "100n" H 9192 2955 50  0000 L CNN
-F 2 "" H 9100 3000 50  0001 C CNN
+F 2 "Capacitor_SMD:C_0603_1608Metric" H 9100 3000 50  0001 C CNN
 F 3 "~" H 9100 3000 50  0001 C CNN
 	1    9100 3000
@@
 F 0 "R4" H 4150 1600 50  0000 L CNN
 F 1 "10k" H 4100 1500 50  0000 L CNN
-F 2 "" H 4300 1550 50  0001 C CNN
+F 2 "Resistor_SMD:R_0603_1608Metric" H 4300 1550 50  0001 C CNN
 F 3 "~" H 4300 1550 50  0001 C CNN
 	1    4300 1550
@@
 F 0 "JP1" V 2804 1248 50  0000 L CNN
 F 1 "Jumper" V 2895 1248 50  0000 L CNN
-F 2 "" H 2850 1200 50  0001 C CNN
+F 2 "Jumper:SolderJumper-2_P1.3mm_Open_Pad1.0x1.5mm" H 2850 1200 50  0001 C CNN
 F 3 "~" H 2850 1200 50  0001 C CNN
 	1    2850 1200
@@
 F 0 "JP2" V 5404 1198 50  0000 L CNN
 F 1 "Jumper" V 5495 1198 50  0000 L CNN
-F 2 "" H 5450 1150 50  0001 C CNN
+F 2 "Jumper:SolderJumper-2_P1.3mm_Open_Pad1.0x1.5mm" H 5450 1150 50  0001 C CNN
 F 3 "~" H 5450 1150 50  0001 C CNN
 	1    5450 1150
@@
 F 0 "JP3" V 7604 1798 50  0000 L CNN
 F 1 "Jumper" V 7695 1798 50  0000 L CNN
-F 2 "" H 7650 1750 50  0001 C CNN
+F 2 "Jumper:SolderJumper-2_P1.3mm_Open_Pad1.0x1.5mm" H 7650 1750 50  0001 C CNN
 F 3 "~" H 7650 1750 50  0001 C CNN
 	1    7650 1750
